File: Schematic/NS73M-Breakout.kicad_pcb (KiCad board)
At the start: 2 copper layers, 17 x 25 mm, 6 parts, among them P1 HEADER, P2 RF_OUT, U1 NS73M, Y1 32.768 kHz

Commit message: Cleaned up schematic, gerber packages, added license and PCB screencaps
Connections:
- net Net-(C1-Pad1) renamed /VCC
- net Net-(P1-Pad3) renamed /TEB
- net Net-(P1-Pad4) renamed /CK
- net Net-(P1-Pad5) renamed /DA
- net Net-(P1-Pad6) renamed /LA
- net Net-(P1-Pad7) renamed /I2C
- net Net-(P1-Pad8) renamed /RIN
- net Net-(P1-Pad9) renamed /LIN
Other:
- net class Default: trace_width 3.35 -> 0.25
